File: Starbie/Starbie.kicad_pcb (KiCad board)
At the start: 2 copper layers, 11 parts, among them J1 Conn_01x04_Pin, J2 Conn_01x08_Pin, SW1 SW_Push, SW2 SW_Push, SW3 SW_Push, SW4 SW_Push, SW5 RotaryEncoder, U1 DHT11, U2 XIAO-ESP32-C3-SMD

Commit message: traces and stuff
Parts:
- added G***: LOGO, assetsHL:Lambda, F.Cu at (99.8, 107.7)
- moved SW3 77.4 mm to (98.5, 139.4)
- moved SW4 72.0 mm to (127.0, 129.4)
- moved J2 48.5 mm to (118.0, 71.0), turned to 0 degrees
- moved R1 31.5 mm to (82.0, 78.5), turned to 180 degrees
- moved SW5 29.0 mm to (126.0, 84.0)
- moved SW2 28.5 mm to (72.5, 120.9)
- moved U1 26.0 mm to (82.0, 70.0)
- moved SW1 23.6 mm to (68.5, 91.4)
- moved H1 20.9 mm to (100.0, 59.5)
- moved J1 17.9 mm to (99.8, 119.7)
- moved U2 17.3 mm to (141.4, 107.4), turned to 0 degrees
Connections:
- U2 pad 1: unconnected-(U2-D0-Pad1)_1 -> /GPIO6
- U2 pad 10: unconnected-(U2-D9/BOOT-Pad10) -> /GPIO7
- U2 pad 7: /GPIO6 -> unconnected-(U2-D6-Pad7)
- U2 pad 8: /GPIO7 -> unconnected-(U2-D7-Pad8)
Routing:
- net GND: track 0.00 -> 292.7 mm
- net /DHT11 DATA: track 0.00 -> 100.4 mm
- net /SDA: track 0.00 -> 91.4 mm
- net +3.3V: track 0.00 -> 91.3 mm
- net /SCL: track 0.00 -> 86.1 mm
- net /GPIO3: track 0.00 -> 82.2 mm
- net /GPIO2: track 0.00 -> 80.6 mm
- net /GPIO10: track 0.00 -> 61.3 mm
- net /GPIO7: track 0.00 -> 43.2 mm
- net /GPIO6: track 0.00 -> 29.2 mm
- net /GPIO8: track 0.00 -> 18.3 mm
Other:
- board outline added: 104.4 x 104.4 mm
- board text added: "CLASSIFIED PROPERTY OF BLACK MESA RESEARCH FACILITY"
- board text added: "LAMBDASSISTANT V1 N0BUDGET HARDWARE INC"

Commit message: updated pcd and add prod files
Parts:
- removed SW4: SW_Push, Button_Switch_Keyboard:SW_Cherry_MX_1.00u_PCB
- added BZ1: Buzzer, Buzzer_Beeper:Buzzer_12x9.5RM7.6, F.Cu at (119.7, 136.0)
- added G***: LOGO, assets:heisenberg, F.Cu at (112.0, 143.0)
- added G***: LOGO, assets:scp, F.Cu at (84.0, 95.0)
- moved R1 2.69 mm to (83.0, 81.0)
- moved J2 1.83 mm to (116.5, 72.0)
- moved U1 1.29 mm to (82.7, 71.1)
Connections:
- net /GPIO6 renamed /GPIO0
- net /GPIO7 renamed /GPIO9
Routing:
- net GND: track 292.7 -> 245.9 mm
- net +3.3V: track 91.3 -> 136.5 mm
- net /GPIO2: track 80.6 -> 104.9 mm
- net /SCL: track 86.1 -> 104.5 mm, vias 0 -> 1
- net /GPIO9: track 43.2 -> 31.3 mm, vias 0 -> 1
- net /SDA: track 91.4 -> 79.6 mm, vias 0 -> 1
- net /GPIO8: track 18.3 -> 29.5 mm
- net /GPIO3: track 82.2 -> 77.7 mm, vias 0 -> 1
- net /GPIO10: track 61.3 -> 62.2 mm
- added copper zone on B.Cu, net GND
- added copper zone on F.Cu, net GND
Other:
- board text added: "LAMBDASSISTANT V1.5 N0BUDGET HARDWARE INC"
- board text removed: "LAMBDASSISTANT V1 N0BUDGET HARDWARE INC"
