File: Starbie/Starbie.kicad_sch (KiCad schematic)
At the start: 11 parts, among them J1 Conn_01x04_Pin, J2 Conn_01x08_Pin, SW1 SW_Push, SW2 SW_Push, SW3 SW_Push, SW4 SW_Push, SW5 RotaryEncoder, U1 DHT11, U2 XIAO-ESP32-C3-SMD

Commit message: traces and stuff
Connections:
- net GPIO6: now also U2.1 (D0); no longer U2.7 (D6)
- net GPIO7: now also U2.10 (D9/BOOT); no longer U2.8 (D7)
Changed lines of the file:
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@@
 	)
 	(no_connect
-		(at 135.89 110.49)
+		(at 135.89 133.35)
 	)
 	(no_connect
@@
 	)
 	(no_connect
-		(at 177.8 125.73)
+		(at 177.8 133.35)
 	)
 	(no_connect
@@
 	(wire
 		(pts
+			(xy 133.35 110.49) (xy 135.89 110.49)
+		)
+		(stroke
+			(width 0)
+			(type default)
+		)
+	)
+	(wire
+		(pts
 			(xy 87.63 111.76) (xy 87.63 114.3)
 		)
@@
 	(wire
 		(pts
+			(xy 180.34 125.73) (xy 177.8 125.73)
+		)
+		(stroke
+			(width 0)
+			(type default)
+		)
+	)
+	(wire
+		(pts
 			(xy 154.94 86.36) (xy 154.94 88.9)
 		)
@@
 	(wire
 		(pts
-			(xy 133.35 133.35) (xy 135.89 133.35)
-		)
-		(stroke
-			(width 0)
-			(type default)
-		)
-	)
-	(wire
-		(pts
 			(xy 99.06 111.76) (xy 101.6 111.76)
 		)
@@
 		(pts
 			(xy 82.55 134.62) (xy 71.12 134.62)
-		)
-		(stroke
-			(width 0)
-			(type default)
-		)
-	)
-	(wire
-		(pts
-			(xy 180.34 133.35) (xy 177.8 133.35)
 		)
 		(stroke
@@
 	)
 	(label "GPIO6"
-		(at 133.35 133.35 180)
+		(at 133.35 110.49 180)
 		(effects
 			(font
@@
 	)
 	(label "GPIO7"
-		(at 180.34 133.35 0)
-		(effects
-			(font
+		(at 180.34 125.73 0)
+		(effects
+			(font

Commit message: updated pcd and add prod files
Parts:
- removed SW4: SW_Push, Button_Switch_Keyboard:SW_Cherry_MX_1.00u_PCB, symbol Switch:SW_Push
- added BZ1: Buzzer, Buzzer_Beeper:Buzzer_12x9.5RM7.6, symbol Device:Buzzer
Connections:
- net GND: now also BZ1.2 (-)
- net GPIO8: now also BZ1.1 (+)
- net GPIO6 renamed GPIO0
- net GPIO7 renamed GPIO9
Other:
- moved on the sheet: H1, SW2
